Commit message: Replace psir with prbt inside files

File: snp_psir_description/urdf/acf_with_grinder/acf_110_01_xs_with_grinder.urdf.xacro (robot description, xacro)
@@ -19,5 +19,5 @@
         <origin xyz="0 0 0" rpy="0 0 0" />
         <geometry>
-          <mesh filename="package://snp_psir_description/meshes/acf_with_grinder/acf_110_01_xs_with_grinder.STL" scale="0.001 0.001 0.001"/>
+          <mesh filename="package://snp_prbt_description/meshes/acf_with_grinder/acf_110_01_xs_with_grinder.STL" scale="0.001 0.001 0.001"/>
         </geometry>
         <material name="">

File: snp_psir_description/urdf/acf_with_grinder/acf_111_04_with_grinder.urdf.xacro (robot description, xacro)
@@ -16,5 +16,5 @@
         <origin xyz="0 0 0" rpy="0 0 0" />
         <geometry>
-          <mesh filename="package://snp_psir_description/meshes/acf_with_grinder/acf_111_04_with_grinder.STL" />
+          <mesh filename="package://snp_prbt_description/meshes/acf_with_grinder/acf_111_04_with_grinder.STL" />
         </geometry>
         <material name="">

File: snp_psir_description/urdf/ensenso.urdf.xacro (robot description, xacro)
@@ -11,5 +11,5 @@
         <origin xyz="0 0 0" rpy="0 0 0" />
         <geometry>
-          <mesh filename="package://snp_psir_description/meshes/ensenso_n35.STL" />
+          <mesh filename="package://snp_prbt_description/meshes/ensenso_n35.STL" />
         </geometry>
         <material name="">

File: snp_psir_description/urdf/snp_psir_demo.urdf.xacro (robot description, xacro)
@@ -1,8 +1,8 @@
 <?xml version="1.0"?>
-<robot xmlns:xacro="http://www.ros.org/wiki/xacro" name="snp_psir_description">
+<robot xmlns:xacro="http://www.ros.org/wiki/xacro" name="snp_prbt_description">
   <xacro:include filename="$(find prbt_support)/urdf/prbt_macro.xacro"/>
-  <xacro:include filename="$(find snp_psir_description)/urdf/prbt_gazebo.xacro"/>
-  <xacro:include filename="$(find snp_psir_description)/urdf/snp_tool.urdf.xacro"/>
-  <xacro:include filename="$(find snp_psir_description)/urdf/psir_table.urdf.xacro"/>
+  <xacro:include filename="$(find snp_prbt_description)/urdf/prbt_gazebo.xacro"/>
+  <xacro:include filename="$(find snp_prbt_description)/urdf/snp_tool.urdf.xacro"/>
+  <xacro:include filename="$(find snp_prbt_description)/urdf/prbt_table.urdf.xacro"/>
   <xacro:property name="prefix" value="prbt_"/>
   <!-- world-->

File: snp_psir_description/urdf/snp_tool.urdf.xacro (robot description, xacro)
@@ -2,6 +2,6 @@
 <robot xmlns:xacro="http://www.ros.org/wiki/xacro">
   <xacro:macro name="snp_tool" params="parent *origin prefix:=${''}">
-    <xacro:include filename="$(find snp_psir_description)/urdf/acf_with_grinder/acf_110_01_xs_with_grinder.urdf.xacro"/>
-    <xacro:include filename="$(find snp_psir_description)/urdf/ensenso.urdf.xacro"/>
+    <xacro:include filename="$(find snp_prbt_description)/urdf/acf_with_grinder/acf_110_01_xs_with_grinder.urdf.xacro"/>
+    <xacro:include filename="$(find snp_prbt_description)/urdf/ensenso.urdf.xacro"/>
     <!-- tool fixture -->
     <link name="${prefix}tool_fixture">
@@ -14,5 +14,5 @@
         <origin xyz="0 0 0" rpy="0 0 0" />
         <geometry>
-          <mesh filename="package://snp_psir_description/meshes/tool_fixture.STL" />
+          <mesh filename="package://snp_prbt_description/meshes/tool_fixture.STL" />
         </geometry>
         <material name="">
@@ -23,5 +23,5 @@
         <origin xyz="0 0 0" rpy="0 0 0" />
         <geometry>
-          <mesh filename="package://snp_psir_description/meshes/tool_fixture.STL" />
+          <mesh filename="package://snp_prbt_description/meshes/tool_fixture.STL" />
         </geometry>
       </collision>
