Commit message: move table down

File: snp_prbt_description/urdf/snp_prbt_demo.urdf.xacro (robot description, xacro)
@@ -15,5 +15,5 @@
   <!-- table-->
   <xacro:table parent="world_frame">
-    <origin  xyz="0 0 0" rpy="0 0 0" />
+    <origin  xyz="0 0 -0.08" rpy="0 0 0" />
   </xacro:table>
   <!-- tool -->
